Commit message: 修复 urdf 文件中 将 base_link 的材质透明度降低，以便看到内部的 imu_link

File: src/fishbot_description/urdf/first_robot.urdf (robot description, URDF)
Before this commit: robot first_robot, 2 links, 1 joints
Links:
- link imu_link: geometry visual box size=0.05 0.05 0.05
Joints:
- joint imu_joint: origin xyz=0 0 0.03 rpy=0 0 0 -> xyz=0 0 0.1 rpy=0 0 0

Commit message: urdf

File: src/fishbot_description/urdf/first_robot.urdf (robot description, URDF)
Before this commit: robot first_robot, 2 links, 1 joints
Links:
- added link camera_link, mass 0.01; collision box size=0.03 0.02 0.02; visual box size=0.03 0.02 0.02
- added link column_link, mass 0.05; collision cylinder length=0.2 radius=0.02; visual cylinder length=0.2 radius=0.02
- added link laser_link, mass 0.01; collision cylinder length=0.04 radius=0.04; visual cylinder length=0.04 radius=0.04
- added link left_arm_link, mass 0.03; collision box size=0.02 0.15 0.02; visual box size=0.02 0.15 0.02
- added link left_hand_link, mass 0.01; collision sphere radius=0.015; visual sphere radius=0.015
- added link odom_link, mass 0.001; collision box size=0.02 0.02 0.02; visual box size=0.02 0.02 0.02
- added link right_arm_link, mass 0.03; collision box size=0.02 0.15 0.02; visual box size=0.02 0.15 0.02
- added link right_hand_link, mass 0.01; collision sphere radius=0.015; visual sphere radius=0.015
- added link wheel_back_left, mass 0.02; collision cylinder length=0.02 radius=0.03; visual cylinder length=0.02 radius=0.03
- added link wheel_back_right, mass 0.02; collision cylinder length=0.02 radius=0.03; visual cylinder length=0.02 radius=0.03
- added link wheel_front_left, mass 0.02; collision cylinder length=0.02 radius=0.03; visual cylinder length=0.02 radius=0.03
- added link wheel_front_right, mass 0.02; collision cylinder length=0.02 radius=0.03; visual cylinder length=0.02 radius=0.03
- link base_link: mass None -> 0.2; geometry collision cylinder length=0.12 radius=0.10; visual cylinder length=0.12 radius=0.10
- link imu_link: mass None -> 0.005; geometry collision box size=0.05 0.05 0.05; visual box size=0.05 0.05 0.05
Joints:
- added joint camera_joint: type fixed, parent column_link, child camera_link, origin xyz=0.06 0 0.15 rpy=0 1.57 0
- added joint column_joint: type fixed, parent base_link, child column_link, origin xyz=0 0 0.12 rpy=0 0 0
- added joint laser_joint: type fixed, parent column_link, child laser_link, origin xyz=0 0 0.2 rpy=0 0 0
- added joint left_hand_joint: type fixed, parent left_arm_link, child left_hand_link, origin xyz=0 -0.075 0 rpy=0 0 0
- added joint left_shoulder_joint: type revolute, parent column_link, child left_arm_link, origin xyz=0 -0.05 0.1 rpy=0 0 0, axis 1 0 0, limit lower=-1.57 upper=1.57 effort=1.0 velocity=0.5
- added joint odom_joint: type fixed, parent base_link, child odom_link, origin xyz=0 0 0 rpy=0 0 0
- added joint right_hand_joint: type fixed, parent right_arm_link, child right_hand_link, origin xyz=0 0.075 0 rpy=0 0 0
- added joint right_shoulder_joint: type revolute, parent column_link, child right_arm_link, origin xyz=0 0.05 0.1 rpy=0 0 0, axis 1 0 0, limit lower=-1.57 upper=1.57 effort=1.0 velocity=0.5
- added joint wheel_bl_joint: type continuous, parent base_link, child wheel_back_left, origin xyz=-0.08485 0.08485 0 rpy=0 0 0, axis 0 1 0
- added joint wheel_br_joint: type continuous, parent base_link, child wheel_back_right, origin xyz=-0.08485 -0.08485 0 rpy=0 0 0, axis 0 1 0
- added joint wheel_fl_joint: type continuous, parent base_link, child wheel_front_left, origin xyz=0.08485 0.08485 0 rpy=0 0 0, axis 0 1 0
- added joint wheel_fr_joint: type continuous, parent base_link, child wheel_front_right, origin xyz=0.08485 -0.08485 0 rpy=0 0 0, axis 0 1 0

Commit message: add gazebo env

File: src/fishbot_description/urdf/first_robot.urdf (robot description, URDF)
Before this commit: robot first_robot, 14 links, 13 joints
Links:
- removed link camera_link
- removed link column_link
- removed link laser_link
- removed link left_arm_link
- removed link left_hand_link
- removed link odom_link
- removed link right_arm_link
- removed link right_hand_link
- removed link wheel_back_left
- removed link wheel_back_right
- removed link wheel_front_left
- removed link wheel_front_right
- link base_link: mass 0.2 -> None; geometry visual cylinder length=0.12 radius=0.10
- link imu_link: mass 0.005 -> None; geometry visual box size=0.05 0.05 0.05
Joints:
- removed joint camera_joint
- removed joint column_joint
- removed joint laser_joint
- removed joint left_hand_joint
- removed joint left_shoulder_joint
- removed joint odom_joint
- removed joint right_hand_joint
- removed joint right_shoulder_joint
- removed joint wheel_bl_joint
- removed joint wheel_br_joint
- removed joint wheel_fl_joint
- removed joint wheel_fr_joint
